File: Cygolite-Clone.kicad_sch (KiCad schematic)
At the start: 33 parts, among them J1 USB4125-GF-A-0190, J2 530480310, J3 Conn_01x03_Socket, J4 Conn_01x02_Socket, SW1 SW_Push, U1 ATtiny202-SS, U2 MCP73831-2-OT, U3 MIC4802YME

Commit message: added v1.0 as built files
Other:
- note added: "@smaroukis"
- title: (none) -> Cygolite Bike Light Clone v1.0
Changed lines of the file:
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@@
 	(generator_version "9.0")
 	(paper "A4")
+	(title_block
+		(title "Cygolite Bike Light Clone v1.0")
+		(date "2026-03-23")
+	)
 	(text "500mA max\nI = 1/Rprog\n"
 		(exclude_from_sim no)
@@
 			)
 		)
+	)
+	(text "@smaroukis"
+		(exclude_from_sim no)
+		(at 250.444 189.484 0)
+		(effects
+			(font
+				(size 2.54 2.54)
+			)
+		)
